Commit message: add 'Joint Controller' and 'RBDL'

File: quadruped_robot_description/urdf/quadruped_robot.urdf (robot description, URDF)
Before this commit: robot qbot, 17 links, 16 joints
Links:
- link BODY: geometry collision box size=0.7 0.230 0.15; visual box size=0.7 0.230 0.15
- link FL_CALF: geometry collision cylinder length=0.309 radius=0.02; visual cylinder length=0.309 radius=0.02
- link FL_HIP: geometry collision cylinder length=0.1 radius=0.05; visual cylinder length=0.1 radius=0.05
- link FL_THIGH: geometry collision cylinder length=0.305 radius=0.02; visual cylinder length=0.305 radius=0.02
- link FR_CALF: geometry collision cylinder length=0.309 radius=0.02; visual cylinder length=0.309 radius=0.02
- link FR_HIP: geometry collision cylinder length=0.1 radius=0.05; visual cylinder length=0.1 radius=0.05
- link FR_THIGH: geometry collision cylinder length=0.309 radius=0.02; visual cylinder length=0.309 radius=0.02
- link RL_CALF: geometry collision cylinder length=0.309 radius=0.02; visual cylinder length=0.309 radius=0.02
- link RL_HIP: geometry collision cylinder length=0.1 radius=0.05; visual cylinder length=0.1 radius=0.05
- link RL_THIGH: geometry collision cylinder length=0.305 radius=0.02; visual cylinder length=0.305 radius=0.02
- link RR_CALF: geometry collision cylinder length=0.309 radius=0.02; visual cylinder length=0.309 radius=0.02
- link RR_HIP: geometry collision cylinder length=0.1 radius=0.05; visual cylinder length=0.1 radius=0.05
- link RR_THIGH: geometry collision cylinder length=0.305 radius=0.02; visual cylinder length=0.305 radius=0.02
Joints:
- removed joint FL_HR_JOINT
- removed joint FR_HR_JOINT
- removed joint RL_HR_JOINT
- removed joint RR_HR_JOINT
- added joint 1_RL_HR_JOINT: type continuous, parent BODY, child RL_HIP, origin xyz=-0.35 0.115 -0.053 rpy=0 0 0, axis 1 0 0
- added joint 2_RR_HR_JOINT: type continuous, parent BODY, child RR_HIP, origin xyz=-0.35 -0.115 -0.053 rpy=0 0 0, axis 1 0 0
- added joint 3_FL_HR_JOINT: type continuous, parent BODY, child FL_HIP, origin xyz=0.35 0.115 -0.053 rpy=0 0 0, axis 1 0 0
- added joint 4_FR_HR_JOINT: type continuous, parent BODY, child FR_HIP, origin xyz=0.35 -0.115 -0.053 rpy=0 0 0, axis 1 0 0
